File: bldc_health/bldc_health.kicad_pcb (KiCad board)
At the start: 2 copper layers, 35.4 x 35.3 mm, 54 parts, among them J1 UART, J2 SERIAL, J3 USB_C_Receptacle_USB2.0_14P, SW1 Reset, SW2 SW_SPDT, U3 AMS1117-3.3, Y1 8MHz CL20pF

Commit message: Preserve current PCB before recheck repairs
Parts:
- J3: footprint Connector_USB:USB_C_Receptacle_Amphenol_124019772112A -> Aerionix_Local:USB-C-16P_ARM-PCB
- moved C3 2.20 mm to (130.8, 127.1)
- moved J3 2.07 mm to (112.3, 105.8)
- moved C15 0.20 mm to (115.2, 118.2)
Routing:
- net /VBUS: track 86.5 -> 41.9 mm, vias 4 -> 2
- net /VDD_STM: track 117.0 -> 72.7 mm, vias 11 -> 9
- net /VDD: track 139.6 -> 114.5 mm, vias 6 -> 7
- net /USB_D+: track 42.2 -> 29.9 mm, vias 4 -> 3
- net /VDDA: track 49.0 -> 41.9 mm, vias 3 -> 2
- net /PA0: track 40.1 -> 35.9 mm
- net /USB_D-: track 33.3 -> 30.7 mm
- net /SWO: track 13.7 -> 15.2 mm
- net Net-(SW2-B): track 37.9 -> 36.5 mm
- net /Reset: track 32.5 -> 33.9 mm
- net Net-(J3-CC2): track 9.29 -> 8.01 mm
- net /Boot0: track 7.78 -> 6.59 mm
- net /HSE_IN: track 32.5 -> 31.5 mm, vias 4 -> 3
- net Net-(J3-CC1): track 5.21 -> 5.87 mm
- net GND: vias 11 -> 12

Commit message: Close PCB connections and resolve routing DRC findings
Parts:
- U4: footprint EasyEDA_Lib:LGA-24_L3.0-W3.0-P0.40-TL -> Aerionix_Local:ICM-40609-D_LGA24_DirectGround
- moved C6 0.25 mm to (114.7, 120.8)
Routing:
- net /SCL_ICM: track 4.59 -> 48.2 mm, vias 1 -> 4
- net /Reset: track 33.9 -> 77.2 mm, vias 3 -> 8
- net /SDA_ASM: track 20.9 -> 36.6 mm, vias 1 -> 3
- net /VDD: track 114.5 -> 116.3 mm
- net /SDA_ICM: track 31.3 -> 30.3 mm
- net /HSE_IN: track 31.5 -> 31.7 mm, vias 3 -> 2
- net GND: vias 12 -> 15
