File: bldc_health/bldc_health.kicad_sch (KiCad schematic)
At the start: 0 parts

Commit message: schematic
Parts:
- added C1, C2: 10u, Capacitor_SMD:C_0603_1608Metric_Pad1.08x0.95mm_HandSolder, symbol Device:C
- added C10, C11, C12, C9: 100nF, Capacitor_SMD:C_0603_1608Metric_Pad1.08x0.95mm_HandSolder, symbol Device:C
- added C13, C5, C6: 100n, symbol Device:C_Small
- added C14: 2.2u, symbol Device:C_Small
- added C15: 10N, symbol Device:C_Small
- added C3, C8: 10uF, Capacitor_SMD:C_0603_1608Metric_Pad1.08x0.95mm_HandSolder, symbol Device:C
- added C4: 100n, Capacitor_SMD:C_0603_1608Metric_Pad1.08x0.95mm_HandSolder, symbol Device:C
- added C7: 10u, symbol Device:C_Small
- added F2: Polyfuse_Small, Fuse:Fuse_0603_1608Metric_Pad1.05x0.95mm_HandSolder, symbol Device:Polyfuse_Small
- added FB2: 120R, Inductor_SMD:L_0603_1608Metric_Pad1.05x0.95mm_HandSolder, symbol Device:FerriteBead_Small
- added J1: USB_C_Receptacle_USB2.0_14P, usb c vikram bhaiya:USB-C-16P, symbol Connector:USB_C_Receptacle_USB2.0_16P
- added JP2: SolderJumper_2_Bridged, Jumper:SolderJumper-2_P1.3mm_Open_RoundedPad1.0x1.5mm, symbol Jumper:SolderJumper_2_Open
- added JP6, JP7: ICM_SJ, symbol Jumper:SolderJumper_3_Open
- added R1, R2: 5k1, Resistor_SMD:R_0603_1608Metric_Pad0.98x0.95mm_HandSolder, symbol Device:R_US
- added R3, R4, R6, R7: 10k, symbol Device:R_Small_US
- added R5: 1k5, Resistor_SMD:R_0603_1608Metric_Pad0.98x0.95mm_HandSolder, symbol Device:R_US
- added U1: (no value), EasyEDA_Lib:UFQFPN-48_L7.0-W7.0-P0.50-TL-EP5.6, symbol EasyEDA_Lib:STM32G491CCU6
- added U2: (no value), EasyEDA_Lib:LGA-14_L3.0-W2.5-P0.50-TL, symbol EasyEDA_Lib:ASM330LHHXTR
- added U3: (no value), EasyEDA_Lib:LGA-24_L3.0-W3.0-P0.40-TL, symbol EasyEDA_Lib:ICM-40609-D
- added U4: AMS1117-3.3, Package_TO_SOT_SMD:SOT-223-3_TabPin2, symbol Regulator_Linear:AMS1117-3.3
Connections:
- new net: JP6.2 (C), U3.9 (SDO/AD0)
- new net: JP7.2 (C), U2.1 (SDO/SA0)
- new net: J1.B5 (CC2), R2.1
- new net: J1.A5 (CC1), R1.1
- new net: J1.A9 (VBUS), J1.B4 (VBUS), J1.B9 (VBUS), J1.VBUS, JP2.1 (A)
- new net GND: C1.2, C10.2, C11.2, C12.2, C13.2, C14.2, C15.1, C2.2, C3.2, C4.2, C5.2, C6.2, C7.2, C8.2, C9.2, J1.A12 (GND), J1.B1 (GND), J1.B12 (GND), J1.GND, J1.S1 (SHIELD), JP6.1 (A), JP7.1 (A), R1.2, R2.2, U1.49 (VSS), U2.2 (MSDA), U2.3 (MSCL), U2.7 (GND), U3.11 (RESV), U3.18 (GND), U3.20 (RESV), U4.1 (GND)
- new net INT1: U2.4 (INT1)
- new net INT2: U2.9 (INT2)
- new net SCL: R4.1, U2.13 (SCL)
- new net SCL_ICM: R7.1, U3.23 (SCL/SCLK)
- new net SDA: R3.2, U2.14 (SDA)
- new net SDA_ICM: R6.2, U3.24 (SDA/SDI/SDIO)
- new net USB_D+: J1.A6 (D+), J1.B6 (D+), R5.1
- new net USB_D-: J1.A7 (D-), J1.B7 (D-)
- new net VBUS: C1.1, JP2.2 (B), U4.3 (VI)
- new net VDD: C13.1, C14.1, C15.2, C2.1, C5.1, C6.1, C7.1, F2.1, JP6.3 (B), JP7.3 (B), R3.1, R4.2, R5.2, R6.1, R7.2, U2.12 (CS), U2.5 (Vdd_IO), U2.8 (Vdd), U3.13 (VDD), U3.22 (nCS), U3.8 (VDDIO), U4.2 (VO)
- new net VDDA: C4.1, FB2.1, U1.21 (VDDA)
- new net VDD_STM: C10.1, C11.1, C12.1, C3.1, C8.1, C9.1, F2.2, FB2.2, U1.1 (VBAT), U1.23 (VDD), U1.35 (VDD), U1.48 (VDD)
- no-connect marks 0 -> 20
Other:
- note added: "ASM330LHHXTR"
- note added: "ICM-40609-D"
- note added: "USB C RECEPTACLE"
Changed lines of the file:
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@@
 	(generator_version "10.0")
 	(paper "A4")
-	(sheet_instances
-		(path "/"
-			(page "1")
-		)
-	)
-	(embedded_fonts no)
-)

Commit message: schematic
Parts:
- removed JP2: SolderJumper_2_Bridged, Jumper:SolderJumper-2_P1.3mm_Open_RoundedPad1.0x1.5mm, symbol Jumper:SolderJumper_2_Open
- added C16, C17: 33p, Capacitor_SMD:C_0603_1608Metric_Pad1.08x0.95mm_HandSolder, symbol Device:C
- added C18: 100nF, Capacitor_SMD:C_0603_1608Metric_Pad1.08x0.95mm_HandSolder, symbol Device:C
- added C19: 100n, Capacitor_SMD:C_0603_1608Metric_Pad1.08x0.95mm_HandSolder, symbol Device:C
- added C20: 1uF, Capacitor_SMD:C_0603_1608Metric_Pad1.08x0.95mm_HandSolder, symbol Device:C
- added D2: 5V LED, LED_SMD:LED_0805_2012Metric_Pad1.15x1.40mm_HandSolder, symbol Device:LED_Small
- added D4: debug_led, LED_SMD:LED_0805_2012Metric_Pad1.15x1.40mm_HandSolder, symbol Device:LED_Small
- added J2: UART, symbol Connector_Generic:Conn_01x02
- added J6: SERIAL, Connector_PinHeader_2.54mm:PinHeader_1x05_P2.54mm_Vertical, symbol Connector_Generic:Conn_01x05
- added R10, R9: 10k, Resistor_SMD:R_0603_1608Metric_Pad0.98x0.95mm_HandSolder, symbol Device:R_US
- added R12: 500, Resistor_SMD:R_0603_1608Metric_Pad0.98x0.95mm_HandSolder, symbol Device:R_US
- added R8: 1k, Resistor_SMD:R_0603_1608Metric_Pad0.98x0.95mm_HandSolder, symbol Device:R_Small_US
- added SW1: SW_SPDT, Button_Switch_THT:SW_Slide-03_Wuerth-WS-SLTV_10x2.5x6.4_P2.54mm, symbol Switch:SW_SPDT
- added SW2: Reset, RESET:SW_TS09-63-25_CUD, symbol Switch:SW_Push
- added Y1: Crystal, Crystal:Crystal_SMD_HC49-SD, symbol Device:Crystal
Connections:
- net SCL is gone; now on net SCL_ASM: R4.1, U2.13 (SCL)
- net SDA is gone; now on net SDA_ASM: R3.2, U2.14 (SDA)
- net GND: now also C16.2, C17.2, C18.1, C19.2, C20.2, D4.1 (K), J6.5 (Pin_5), R12.2, SW1.1 (A), SW2.2
- net INT1: now also U1.15 (PA7)
- net INT2: now also U1.16 (PC4)
- net SCL_ICM: now also U1.38 (PA15)
- net SDA_ICM: now also U1.45 (PB7)
- net USB_D+: now also U1.34 (PA12)
- net USB_D-: now also U1.33 (PA11)
- net VBUS: now also J1.A9 (VBUS), J1.B4 (VBUS), J1.B9 (VBUS), J1.VBUS, D2.2 (A)
- net VDD: now also J6.1 (Pin_1), R10.2, SW1.3 (C)
- net VDDA: now also U1.20 (VREF+), C19.1, C20.1
- net PA2_TX: now reaches U1.10 (PA2)
- net PA2_TX: now also J2.1 (Pin_1)
- net PA3_RX: now reaches U1.11 (PA3)
- net PA3_RX: now also J2.2 (Pin_2)
- net PB0_INT1_ICM: now reaches U1.17 (PB0)
- net PB0_INT1_ICM: now also U3.12 (INT1/INT)
- net FSYNC: now reaches U1.18 (PB1)
- net FSYNC: now also U3.19 (NT2/FSYNC)
- net PB2: now reaches U1.19 (PB2)
- net PB2: now also R8.2
- net SCL_ASM: now reaches U1.30 (PA8)
- net SWDIO: now reaches U1.36 (PA13)
- net SWDIO: now also J6.2 (Pin_2)
- net SWCLK: now reaches U1.37 (PA14)
- net SWCLK: now also J6.3 (Pin_3)
- net SDA_ASM: now reaches U1.40 (PC11)
- net SWO: now reaches U1.41 (PB3)
- net SWO: now also J6.4 (Pin_4)
- net Boot0: now reaches U1.46 (PB8-BOOT0)
- net Boot0: now also R9.2
- net HSE_IN: now reaches U1.5 (PF0-OSC_IN)
- net HSE_IN: now also C16.1, Y1.1
- net HSE_OUT: now reaches U1.6 (PF1-OSC_OUT)
- net HSE_OUT: now also C17.1, Y1.2
- net Reset: now reaches U1.7 (PG10-NRST)
- net Reset: now also C18.2, R10.1, SW2.1
- new net: D2.1 (K), R12.1
- new net: R9.1, SW1.2 (B)
- new net: D4.2 (A), R8.1
- no-connect marks 20 -> 18
Other:
- note added: "CRYSTAL OSCILLATOR"
- note added: "PWR LED"
- note added: "STM32G491CCU6"
- moved on the sheet: C1, C10, C11, C12, C2, C3, C4, C5, C6, C7, C8, C9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

Commit message: changes to pins
Parts:
- C13, C14, C15, C5, C6, C7: footprint (none) -> Capacitor_SMD:C_0603_1608Metric_Pad1.08x0.95mm_HandSolder
- R3, R4, R6, R7: footprint (none) -> Resistor_SMD:R_0603_1608Metric_Pad0.98x0.95mm_HandSolder
Connections:
- net SCL_ASM: now also U1.31 (PA9); no longer U1.30 (PA8)
- net SDA_ASM: now also U1.30 (PA8); no longer U1.40 (PC11)

Commit message: Update PCB layout and schematic
Parts:
- added R6, Thermistor1: 10k, Resistor_SMD:R_0603_1608Metric_Pad0.98x0.95mm_HandSolder, symbol Device:R_US
- renumbered C19 to C1, C4 to C10, C9 to C11, C3 to C12, C10 to C13, C11 to C14, C12 to C15, C1 to C16, C2 to C17, C15 to C18, C13 to C19, C5 to C2, C14 to C20, C6 to C3, C16 to C4, C7 to C5, C17 to C6, C20 to C7, C18 to C9, D2 to D1, D4 to D2, F2 to F1, FB2 to FB1, J2 to J1, J6 to J2, J1 to J3, JP7 to JP1, JP6 to JP2, R12 to R1, R7 to R10, R1 to R11, R2 to R12, R8 to R2, R10 to R5, R9 to R7, R5 to R8, R6 to R9, SW2 to SW1, SW1 to SW2, U4 to U3, U3 to U4
Connections:
- net GND: now also Thermistor1.2
- net VDDA: now also R6.1
- net PA0: now reaches U1.8 (PA0)
- net PA0: now also R6.2, Thermistor1.1
Other:
- note added: "10k Thermistor"

Commit message: Update PCB layout, footprints, and schematic
Parts:
- J1: footprint (none) -> Connector_PinHeader_2.54mm:PinHeader_1x02_P2.54mm_Vertical
- J3: footprint usb c vikram bhaiya:USB-C-16P -> Connector_USB:USB_C_Receptacle_Amphenol_12401548E4-2A
- JP1, JP2: footprint (none) -> Jumper:SolderJumper-3_P1.3mm_Open_Pad1.0x1.5mm
- SW1: footprint RESET:SW_TS09-63-25_CUD -> TS09-63-25-WT-160-SMT-TR:SW_TS09-63-25-WT-160-SMT-TR
- Thermistor1: footprint Resistor_SMD:R_0603_1608Metric_Pad0.98x0.95mm_HandSolder -> Connector_PinHeader_1.00mm:PinHeader_1x02_P1.00mm_Vertical

Commit message: Apply verified PCB review fixes before USB footprint replacement
Parts:
- added C21: 100nF, Capacitor_SMD:C_0402_1005Metric, symbol Device:C_Small
- J3: footprint Connector_USB:USB_C_Receptacle_Amphenol_12401548E4-2A -> Connector_USB:USB_C_Receptacle_Amphenol_124019772112A
- Y1: value Crystal -> 8MHz CL20pF
Connections:
- net GND: now also J3.A1 (GND), J3.SH (SHIELD), C21.2; no longer J3.GND, J3.S1 (SHIELD)
- net VBUS: now also J3.A4 (VBUS); no longer J3.VBUS
- net VDD: now also C21.1
Other:
- note added: "U2 local bypass; I2C target 100 kHz"

Commit message: Preserve current PCB before recheck repairs
Parts:
- J3: footprint Connector_USB:USB_C_Receptacle_Amphenol_124019772112A -> Aerionix_Local:USB-C-16P_ARM-PCB
Connections:
- net GND: now also J3.GND; no longer J3.A1 (GND), J3.A12 (GND), J3.B1 (GND), J3.B12 (GND)
- net VBUS: now also J3.VBUS; no longer J3.A4 (VBUS), J3.A9 (VBUS), J3.B4 (VBUS), J3.B9 (VBUS)

Commit message: Close PCB connections and resolve routing DRC findings
Parts:
- U4: footprint EasyEDA_Lib:LGA-24_L3.0-W3.0-P0.40-TL -> Aerionix_Local:ICM-40609-D_LGA24_DirectGround
